File: pcb3/pcb3.brd (EAGLE design)
At the start: 101.6 x 53.3 mm, 31 parts, among them J1 12V, J2 24V, J3 RTD, J4 RTD, J5 VFS, J6 RELAY, J7 BRAKES, Q1 BSS314PEH6327XTSA1, Q2 BSS314PEH6327XTSA1, Q3 MMBT2222AT-7-F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

Commit message: Add Serial CAN Bus to PCB 3
Parts:
- added J8: CANBUS, Molex Micro-Lock PLUS:4PIN
- C1, C2: device Capacitor:CAPC1608X85 -> Capacitor:CAPC3216X135
- Q1, Q2: value BSS314PEH6327XTSA1 -> SI01P10-TP
- R1, R2: value (none) -> 150
- R3, R4: value (none) -> 15
- moved C2 1.87 mm to (31.3, 11.9), turned to 180 degrees
Connections:
- removed net 5V: U$1.5V
- new net +5V: J8.1, U$1.5V
- new net N$19: J8.3, U$1.D1
- new net N$20: J8.4, U$1.D0
- net GND: now also J8.2
Routing:
- net +5V: track 0.00 -> 84.2 mm, vias 0 -> 1
- net N$19: track 0.00 -> 35.9 mm
- net N$20: track 0.00 -> 32.9 mm
- net GND: track 71.1 -> 76.0 mm, vias 11 -> 12
- net +12V: track 153.4 -> 155.2 mm
- net +24V: track 63.1 -> 62.4 mm
